Commit message: working learning with pytorch and ppo

File: myGym/envs/objects/geometric/urdf/rectangle.urdf (robot description, URDF)
Before this commit: robot rectangle.urdf, 1 links, 0 joints
Links:
- link baseLink: geometry collision mesh filename=./obj/cube.obj scale=.001 .001 .005; visual mesh filename=./obj/cube.obj scale=.001 .001 .005

File: myGym/envs/objects/geometric/urdf/supercube.urdf (robot description, URDF)
Before this commit: robot supercube.urdf, 2 links, 1 joints
Links:
- link heavierCube: mass 2 -> 10
