Commit message: fixed supercube, started new reward function

File: myGym/envs/objects/geometric/urdf/supercube.urdf (robot description, URDF)
Before this commit: robot supercube.urdf, 2 links, 1 joints
Links:
- removed link baseLink
- removed link heavierCube
- added link base_link, mass 1.0; collision mesh filename=obj/supercube.obj scale=.0021 .0021 .0021; visual mesh filename=obj/supercube.obj scale=.0021 .0021 .0021
- added link heavier_cube, mass 1.13; collision mesh filename=obj/cube.obj scale=.0007 .0007 .0007; visual mesh filename=obj/cube.obj scale=.0007 .0007 .0007
Joints:
- removed joint heavierCubeJoint
- added joint heavier_cube_joint: type fixed, parent base_link, child heavier_cube, origin xyz=0 0 0 rpy=0 0 0
