Commit message: colored cube

File: myGym/envs/objects/geometric/urdf/cube.urdf (robot description, URDF)
Before this commit: robot cube.urdf, 1 links, 0 joints
Links:
- link baseLink: mass 0.113 -> 1.0; geometry collision mesh filename=./obj/cube.obj scale=.1 .1 .1; visual mesh filename=./obj/cube.obj scale=0.1 0.1 0.1

File: myGym/envs/objects/geometric/urdf/rectangle.urdf (robot description, URDF)
Before this commit: robot rectangle.urdf, 1 links, 0 joints
Links:
- link baseLink: geometry collision mesh filename=./obj/rectangle.obj scale=.001 .001 .005; visual mesh filename=./obj/rectangle.obj scale=.001 .001 .005

File: myGym/envs/objects/geometric/urdf/supercube.urdf (robot description, URDF)
Before this commit: robot supercube, 2 links, 1 joints
Links:
- link base_link: mass 1.0 -> 0.1; geometry collision mesh filename=../obj/supercube.obj scale=.0021 .0021 .0021; visual mesh filename=../obj/supercube.obj scale=.0021 .0021 .0021
- link heavier_cube: mass 1.13 -> 0.1; geometry collision mesh filename=../obj/cube.obj scale=.0007 .0007 .0007; visual mesh filename=../obj/cube.obj scale=.0007 .0007 .0007

Commit message: updated, working com loss and training, potentially needs tuning

File: myGym/envs/objects/geometric/urdf/cube.urdf (robot description, URDF)
Before this commit: robot cube.urdf, 1 links, 0 joints
Links:
- link baseLink: mass 1.0 -> 0.5

Commit message: more stable config, less flailing

File: myGym/envs/objects/geometric/urdf/cube.urdf (robot description, URDF)
Before this commit: robot cube.urdf, 1 links, 0 joints
Links:
- link baseLink: mass 0.5 -> 1

Commit message: method_2_approach
These are the changes made for the Method 2

File: myGym/envs/objects/geometric/urdf/cube.urdf (robot description, URDF)
Before this commit: robot cube.urdf, 1 links, 0 joints
Links:
- link baseLink: mass 1.0 -> 0.1

File: myGym/envs/objects/geometric/urdf/obj_temp.urdf (robot description, URDF)
Before this commit: robot cube.urdf, 1 links, 0 joints
Links:
- link baseLink: mass 1.0 -> 0.1
